Commit message: ultimate fix?

File: resources/T1/T1_serial.urdf (robot description, URDF)
Before this commit: robot T1, 24 links, 23 joints
Joints:
- joint AAHead_yaw: type revolute -> fixed
- joint Head_pitch: type revolute -> fixed

Commit message: no more t pose

File: resources/T1/T1_serial.urdf (robot description, URDF)
Before this commit: robot T1, 24 links, 23 joints
Joints:
- joint Left_Elbow_Yaw: origin xyz=0 0.1471 0 rpy=0 0 0 -> xyz=0 0.1471 0 rpy=0 0 -0.5
- joint Left_Shoulder_Pitch: origin xyz=0.0575 0.1063 0.219 rpy=0 0.00088113 0 -> xyz=0.0575 0.1063 0.219 rpy=0 0.2 0
- joint Left_Shoulder_Roll: origin xyz=0 0.047 0 rpy=0 0 0 -> xyz=0 0.047 0 rpy=-1.35 0 0
- joint Right_Elbow_Yaw: origin xyz=0 -0.1471 0 rpy=0 0 0 -> xyz=0 -0.1471 0 rpy=0 0 0.5
- joint Right_Shoulder_Pitch: origin xyz=0.0575 -0.1063 0.219 rpy=0 0.00088113 0 -> xyz=0.0575 -0.1063 0.219 rpy=0 0.2 0
- joint Right_Shoulder_Roll: origin xyz=0 -0.047 0 rpy=0 0 0 -> xyz=0 -0.047 0 rpy=1.35 0 0
