Commit message: adding arms

File: resources/T1/T1_locomotion.urdf (robot description, URDF)
Before this commit: robot T1, 24 links, 23 joints
Joints:
- joint Left_Elbow_Pitch: type fixed -> revolute
- joint Left_Elbow_Yaw: type fixed -> revolute
- joint Left_Shoulder_Pitch: type fixed -> revolute
- joint Left_Shoulder_Roll: type fixed -> revolute
- joint Right_Elbow_Pitch: type fixed -> revolute
- joint Right_Elbow_Yaw: type fixed -> revolute
- joint Right_Shoulder_Pitch: type fixed -> revolute
- joint Right_Shoulder_Roll: type fixed -> revolute
- joint Waist: type fixed -> revolute

Commit message: added constraints to shoulder and elbow

File: resources/T1/T1_locomotion.urdf (robot description, URDF)
Before this commit: robot T1, 24 links, 23 joints
Joints:
- joint Left_Elbow_Yaw: type revolute -> fixed
- joint Left_Shoulder_Roll: type revolute -> fixed
- joint Right_Elbow_Yaw: type revolute -> fixed
- joint Right_Shoulder_Roll: type revolute -> fixed

Commit message: changes

File: resources/T1/T1_locomotion.urdf (robot description, URDF)
Before this commit: robot T1, 24 links, 23 joints
Joints:
- joint Left_Elbow_Yaw: type fixed -> revolute
- joint Left_Shoulder_Roll: type fixed -> revolute
- joint Right_Elbow_Yaw: type fixed -> revolute
- joint Right_Shoulder_Roll: type fixed -> revolute

Commit message: adding collissions to the arms

File: resources/T1/T1_locomotion.urdf (robot description, URDF)
Before this commit: robot T1, 24 links, 23 joints
Links:
- link AL1: geometry collision capsule length=0.047 radius=0.04; visual mesh filename=meshes/AL1.STL
- link AL2: geometry collision capsule length=0.0605 radius=0.04; visual mesh filename=meshes/AL2.STL
- link AL3: geometry collision capsule length=0.1471 radius=0.04; visual mesh filename=meshes/AL3.STL
- link AR1: geometry collision capsule length=0.047 radius=0.04; visual mesh filename=meshes/AR1.STL
- link AR2: geometry collision capsule length=0.0605 radius=0.04; visual mesh filename=meshes/AR2.STL
- link AR3: geometry collision capsule length=0.1471 radius=0.04; visual mesh filename=meshes/AR3.STL
- link Ankle_Cross_Left: geometry collision capsule length=0.012 radius=0.02; visual mesh filename=meshes/Ankle_Cross_Left.STL
- link Ankle_Cross_Right: geometry collision capsule length=0.012 radius=0.02; visual mesh filename=meshes/Ankle_Cross_Right.STL
- link H1: geometry collision capsule length=0.06185 radius=0.03; visual mesh filename=meshes/H1.STL
- link H2: geometry collision sphere radius=0.06; visual mesh filename=meshes/H2.STL
- link Hip_Pitch_Left: geometry collision capsule length=0.02 radius=0.04; visual mesh filename=meshes/Hip_Pitch_Left.STL
- link Hip_Pitch_Right: geometry collision capsule length=0.02 radius=0.04; visual mesh filename=meshes/Hip_Pitch_Right.STL
- link Hip_Roll_Left: geometry collision capsule length=0.081854 radius=0.04; visual mesh filename=meshes/Hip_Roll_Left.STL
- link Hip_Roll_Right: geometry collision capsule length=0.081854 radius=0.04; visual mesh filename=meshes/Hip_Roll_Right.STL
- link Waist: geometry collision cylinder length=0.1 radius=0.11; visual mesh filename=meshes/Waist.STL
- link left_hand_link: geometry collision sphere radius=0.04; visual mesh filename=meshes/left_hand_link.STL
- link right_hand_link: geometry collision sphere radius=0.04; visual mesh filename=meshes/right_hand_link.STL

Commit message: delete collisions of arms

File: resources/T1/T1_locomotion.urdf (robot description, URDF)
Before this commit: robot T1, 24 links, 23 joints
Links:
- link AL1: geometry visual mesh filename=meshes/AL1.STL
- link AL2: geometry visual mesh filename=meshes/AL2.STL
- link AL3: geometry visual mesh filename=meshes/AL3.STL
- link AR1: geometry visual mesh filename=meshes/AR1.STL
- link AR2: geometry visual mesh filename=meshes/AR2.STL
- link AR3: geometry visual mesh filename=meshes/AR3.STL
- link Ankle_Cross_Left: geometry visual mesh filename=meshes/Ankle_Cross_Left.STL
- link Ankle_Cross_Right: geometry visual mesh filename=meshes/Ankle_Cross_Right.STL
- link H1: geometry visual mesh filename=meshes/H1.STL
- link H2: geometry visual mesh filename=meshes/H2.STL
- link Hip_Pitch_Left: geometry visual mesh filename=meshes/Hip_Pitch_Left.STL
- link Hip_Pitch_Right: geometry visual mesh filename=meshes/Hip_Pitch_Right.STL
- link Hip_Roll_Left: geometry visual mesh filename=meshes/Hip_Roll_Left.STL
- link Hip_Roll_Right: geometry visual mesh filename=meshes/Hip_Roll_Right.STL
- link Waist: geometry visual mesh filename=meshes/Waist.STL
- link left_hand_link: geometry visual mesh filename=meshes/left_hand_link.STL
- link right_hand_link: geometry visual mesh filename=meshes/right_hand_link.STL

Commit message: adding hand collisions

File: resources/T1/T1_locomotion.urdf (robot description, URDF)
Before this commit: robot T1, 24 links, 23 joints
Links:
- link left_hand_link: geometry collision mesh filename=meshes/left_hand_link.STL; visual mesh filename=meshes/left_hand_link.STL
- link right_hand_link: geometry collision mesh filename=meshes/right_hand_link.STL; visual mesh filename=meshes/right_hand_link.STL

Commit message: resetting to locomotion

File: resources/T1/T1_locomotion.urdf (robot description, URDF)
Before this commit: robot T1, 24 links, 23 joints
Links:
- link left_hand_link: geometry visual mesh filename=meshes/left_hand_link.STL
- link right_hand_link: geometry visual mesh filename=meshes/right_hand_link.STL
